File: ControllerBoxSTM32F401.kicad_sch (KiCad schematic)
At the start: 56 parts, among them SW1 Switch, SW10 Switch, SW11 Switch, SW12 Switch, SW13 Switch, SW14 Switch, SW15 Switch, SW16 Switch, SW17 Switch, SW18 Switch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

Commit message: update PCB and create edge cuts
Parts:
- C1, C2, C3, C4, C5, C6: footprint Capacitor_THT:C_Disc_D5.0mm_W2.5mm_P5.00mm -> Capacitor_THT:C_Radial_D6.3mm_H7.0mm_P2.50mm
- G29SHIFTER1: value DB9_Female -> DB9_Male; footprint Connector_Dsub:DSUB-9_Female_Horizontal_P2.77x2.84mm_EdgePinOffset4.94mm_Housed_MountingHolesOffset7.48mm -> Connector_Dsub:DSUB-9_Male_Horizontal_P2.77x2.84mm_EdgePinOffset7.70mm_Housed_MountingHolesOffset9.12mm
Connections:
- net GND: now also U1.19 (GND)
- net VCC 3.3V: now also U1.20 (3V3)
- net VCC 5V: now also U1.18 (5V)
- no-connect marks 32 -> 29
Changed lines of the file:
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@@
   (no_connect (at 101.6 87.63))
   (no_connect (at 101.6 90.17))
-  (no_connect (at 101.6 97.79))
-  (no_connect (at 101.6 102.87))
-  (no_connect (at 101.6 100.33))
   (no_connect (at 147.32 102.87))
   (no_connect (at 147.32 100.33))
@@
     )
   )
+  (global_label "VCC 3.3V" (shape input) (at 101.6 102.87 180) (fields_autoplaced)
+    (effects (font (size 1 1)) (justify right))
+    (property "Intersheet References" "${INTERSHEET_REFS}" (id 0) (at 92.8429 102.9325 0)
+      (effects (font (size 1 1)) (justify right) hide)
+    )
+  )
   (global_label "BTN_COL3" (shape input) (at 147.32 97.79 0) (fields_autoplaced)
     (effects (font (size 1.27 1.27)) (justify left))
@@
     (property "Intersheet References" "${INTERSHEET_REFS}" (id 0) (at 189.7683 62.3094 0)
       (effects (font (size 1.27 1.27)) (justify left) hide)
+    )
+  )
+  (global_label "VCC 5V" (shape input) (at 101.6 97.79 180) (fields_autoplaced)
+    (effects (font (size 1 1)) (justify right))
+    (property "Intersheet References" "${INTERSHEET_REFS}" (id 0) (at 94.2714 97.8525 0)
+      (effects (font (size 1 1)) (justify right) hide)
     )
   )
@@
     )
   )
+  (global_label "GND" (shape input) (at 101.6 100.33 180) (fields_autoplaced)
+    (effects (font (size 1 1)) (justify right))
+    (property "Intersheet References" "${INTERSHEET_REFS}" (id 0) (at 96.6524 100.3925 0)
+      (effects (font (size 1 1)) (justify right) hide)
+    )
+  )
   (global_label "ENC B" (shape input) (at 179.07 87.63 0) (fields_autoplaced)
     (effects (font (size 0.8 0.8)) (justify left))
@@
       (effects (font (size 1.27 1.27)) (justify left))
     )
-    (property "Footprint" "Capacitor_THT:C_Disc_D5.0mm_W2.5mm_P5.00mm" (id 2) (at 176.2252 69.85 0)
+    (property "Footprint" "Capacitor_THT:C_Radial_D6.3mm_H7.0mm_P2.50mm" (id 2) (at 176.2252 69.85 0)
       (effects (font (size 1.27 1.27)) hide)
     )
@@
       (effects (font (size 1.27 1.27)) (justify left) hide)
     )
-    (property "Footprint" "Capacitor_THT:C_Disc_D5.0mm_W2.5mm_P5.00mm" (id 2) (at 160.9852 80.01 0)
+    (property "Footprint" "Capacitor_THT:C_Radial_D6.3mm_H7.0mm_P2.50mm" (id 2) (at 160.9852 80.01 0)
       (effects (font (size 1.27 1.27)) hide)
     )
@@
       (effects (font (size 1.27 1.27)) (justify left) hide)
     )
-    (property "Footprint" "Capacitor_THT:C_Disc_D5.0mm_W2.5mm_P5.00mm" (id 2) (at 164.7952 77.47 0)
+    (property "Footprint" "Capacitor_THT:C_Radial_D6.3mm_H7.0mm_P2.50mm" (id 2) (at 164.7952 77.47 0)
       (effects (font (size 1.27 1.27)) hide)
     )
@@
       (effects (font (size 1.27 1.27)) (justify left))
     )
-    (property "Value" "DB9_Female" (id 1) (at 259.08 126.9999 0)
-      (effects (font (size 1.27 1.27)) (justify left))
-    )
-    (property "Footprint" "Connector_Dsub:DSUB-9_Female_Horizontal_P2.77x2.84mm_EdgePinOffset4.94mm_Housed_MountingHolesOffset7.48mm" (id 2) (at 254 125.73 0)
+    (property "Value" "DB9_Male" (id 1) (at 259.08 126.9999 0)
+      (effects (font (size 1.27 1.27)) (justify left))
+    )
+    (property "Footprint" "Connector_Dsub:DSUB-9_Male_Horizontal_P2.77x2.84mm_EdgePinOffset7.70mm_Housed_MountingHolesOffset9.12mm" (id 2) (at 254 125.73 0)
       (effects (font (size 1.27 1.27)) hide)
     )
@@
       (effects (font (size 1.27 1.27)) (justify left) hide)
     )
-    (property "Footprint" "Capacitor_THT:C_Disc_D5.0mm_W2.5mm_P5.00mm" (id 2) (at 172.4152 72.39 0)
+    (property "Footprint" "Capacitor_THT:C_Radial_D6.3mm_H7.0mm_P2.50mm" (id 2) (at 172.4152 72.39 0)
       (effects (font (size 1.27 1.27)) hide)
     )
@@
       (effects (font (size 1.27 1.27)) (justify left) hide)
     )
-    (property "Footprint" "Capacitor_THT:C_Disc_D5.0mm_W2.5mm_P5.00mm" (id 2) (at 168.6052 74.93 0)
+    (property "Footprint" "Capacitor_THT:C_Radial_D6.3mm_H7.0mm_P2.50mm" (id 2) (at 168.6052 74.93 0)
       (effects (font (size 1.27 1.27)) hide)
     )
@@
       (effects (font (size 1.27 1.27)) (justify right) hide)
     )
-    (property "Footprint" "Capacitor_THT:C_Disc_D5.0mm_W2.5mm_P5.00mm" (id 2) (at 155.2448 74.93 0)
+    (property "Footprint" "Capacitor_THT:C_Radial_D6.3mm_H7.0mm_P2.50mm" (id 2) (at 155.2448 74.93 0)
       (effects (font (size 1.27 1.27)) hide)
     )
@@
   (symbol_instances
     (path "/b09ebe36-1317-4319-9481-e171f85671e1"
-      (reference "C1") (unit 1) (value "10uF") (footprint "Capacitor_THT:C_Disc_D5.0mm_W2.5mm_P5.00mm")
+      (reference "C1") (unit 1) (value "10uF") (footprint "Capacitor_THT:C_Radial_D6.3mm_H7.0mm_P2.50mm")
     )
     (path "/2bcd5d0d-c36e-4bdf-9835-5401928b4417"
-      (reference "C2") (unit 1) (value "10uF") (footprint "Capacitor_THT:C_Disc_D5.0mm_W2.5mm_P5.00mm")
+      (reference "C2") (unit 1) (value "10uF") (footprint "Capacitor_THT:C_Radial_D6.3mm_H7.0mm_P2.50mm")
     )
     (path "/479efe71-3a1e-4ee9-bfdb-f65aff1d125e"
-      (reference "C3") (unit 1) (value "10uF") (footprint "Capacitor_THT:C_Disc_D5.0mm_W2.5mm_P5.00mm")
+      (reference "C3") (unit 1) (value "10uF") (footprint "Capacitor_THT:C_Radial_D6.3mm_H7.0mm_P2.50mm")
     )
     (path "/9f966eb3-c911-4c44-a893-c9aafd674e66"
-      (reference "C4") (unit 1) (value "10uF") (footprint "Capacitor_THT:C_Disc_D5.0mm_W2.5mm_P5.00mm")
+      (reference "C4") (unit 1) (value "10uF") (footprint "Capacitor_THT:C_Radial_D6.3mm_H7.0mm_P2.50mm")
     )
     (path "/83fe9231-d52f-4b2e-8cdd-09ea427ee499"
-      (reference "C5") (unit 1) (value "10uF") (footprint "Capacitor_THT:C_Disc_D5.0mm_W2.5mm_P5.00mm")
+      (reference "C5") (unit 1) (value "10uF") (footprint "Capacitor_THT:C_Radial_D6.3mm_H7.0mm_P2.50mm")
     )
     (path "/14d1528a-149b-4a66-8893-984d709a281a"
-      (reference "C6") (unit 1) (value "10uF") (footprint "Capacitor_THT:C_Disc_D5.0mm_W2.5mm_P5.00mm")
+      (reference "C6") (unit 1) (value "10uF") (footprint "Capacitor_THT:C_Radial_D6.3mm_H7.0mm_P2.50mm")
     )
     (path "/4cd1982f-4ec5-4b04-b58d-47b3d64201c1"
@@
     )
     (path "/7e80398f-b27e-4d8e-ba77-b4cae8b32463"
-      (reference "G29SHIFTER1") (unit 1) (value "DB9_Female") (footprint "Connector_Dsub:DSUB-9_Female_Horizontal_P2.77x2.84mm_EdgePinOffset4.94mm_Housed_MountingHolesOffset7.48mm")
+      (reference "G29SHIFTER1") (unit 1) (value "DB9_Male") (footprint "Connector_Dsub:DSUB-9_Male_Horizontal_P2.77x2.84mm_EdgePinOffset7.70mm_Housed_MountingHolesOffset9.12mm")
     )
     (path "/521ba1cd-b851-4321-9308-4f6311c86448"

Commit message: add button matrix to PCB
Parts:
- removed D1, D10, D11, D12, D13, D14, D15, D16, D2, D3, D4, D5, D6, D7, D8, D9: D, symbol Device:D
- added D1, D10, D11, D12, D13, D14, D15, D16, D2, D3, D4, D5, D6, D7, D8, D9: 1N4148, Diode_THT:D_DO-35_SOD27_P7.62mm_Horizontal, symbol Diode:1N4148
- HBRAKE1, PEDAL1, STEERINGWHEEL1: footprint RJ45_Hanrun_HR911105A -> Connector_RJ:RJ45_Ninigi_GE
- SW1, SW10, SW11, SW12, SW13, SW14, SW15, SW16, SW17, SW18, SW19, SW2, SW20, SW3, SW4, SW5, SW6, SW7, SW8, SW9: footprint (none) -> Connector_PinHeader_2.54mm:PinHeader_1x02_P2.54mm_Vertical
Connections:
- net BTN_COL1: now also SW6.1, D1.1 (K); no longer SW2.1
- net BTN_COL2: now also SW11.1, SW6.2, D5.1 (K); no longer SW2.2, SW3.1
- net BTN_COL3: now also SW11.2, SW16.1, D9.1 (K); no longer SW3.2, SW4.1
- net BTN_COL4: now also SW16.2, D13.1 (K); no longer SW4.2
- net BTN_ROW2: now also SW2.1; no longer SW5.1
- net BTN_ROW3: now also SW3.1; no longer SW9.1
- net BTN_ROW4: now also SW4.1; no longer SW13.1
- net BTN_ROW5: now also SW5.1; no longer SW17.1
- net at SW7.1: now also SW2.2, D1.2 (A), D2.1 (K); no longer SW6.2
- net at SW10.2: now also SW15.1, D8.2 (A); no longer SW11.1
- net at SW19.1: now also SW14.2, D11.2 (A), D12.1 (K); no longer SW18.2
- net at SW19.2: now also D15.2 (A), D16.1 (K); no longer SW20.1
- net at SW7.2: now also SW12.1, D5.2 (A), D6.1 (K); no longer SW8.1
- net at SW8.2: now also SW13.1, D6.2 (A), D7.1 (K)
- net at SW5.2: now also SW10.1, D4.2 (A); no longer SW6.1
- net at SW12.2: now also SW17.1, D10.1 (K), D9.2 (A)
- net at SW15.2: now also SW20.1, D12.2 (A); no longer SW16.1
- net at SW13.2: now also SW18.1, D10.2 (A), D11.1 (K); no longer SW14.1
- net at SW17.2: now also D13.2 (A), D14.1 (K); no longer SW18.1
- net at SW9.2: now also SW14.1, D7.2 (A), D8.1 (K); no longer SW10.1
- net at SW20.2: now also D16.2 (A)
- new net: D3.2 (A), D4.1 (K), SW4.2, SW9.1
- new net: D2.2 (A), D3.1 (K), SW3.2, SW8.1
- new net: D14.2 (A), D15.1 (K), SW18.2
