File: ControllerBoxSTM32F401.kicad_pcb (KiCad board)
At the start: 2 copper layers, 62.4 x 75.6 mm, 22 parts, among them J1 ROW BUTTON, J2 COL BUTTON, U1 YAAJ_WeAct_BlackPill_Part_Lik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

Commit message: update pcb production
Routing:
- net VCC 5V: track 45.1 -> 95.4 mm
- net Net-(R6-Pad2): track 0.00 -> 11.4 mm
- net Net-(R4-Pad2): track 0.00 -> 6.68 mm, vias 0 -> 1
- net ACCEL: track 15.4 -> 21.6 mm
- net Net-(R5-Pad2): track 0.00 -> 5.47 mm
- net CLUTCH: track 15.4 -> 16.3 mm
Other:
- board text added: "10uF"
- board text added: "220"
- board text added: "4.7k"
- board text added: "ControllerBox STM32F4x1 EMCPro Firmware (c) Rockavoldy 2022"
Changed lines of the file:
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@@
     (pad_to_mask_clearance 0)
     (pcbplotparams
-      (layerselection 0x00010fc_ffffffff)
+      (layerselection 0x00210fc_ffffffff)
       (disableapertmacros false)
       (usegerberextensions false)
@@
       (effects (font (size 1 1) (thickness 0.15)))
     )
-    (fp_text user "${REFERENCE}" (at 0 0) (layer "F.Fab")
-      (effects (font (size 0.5 0.5) (thickness 0.08)))
+    (fp_text user "${REFERENCE}" (at 0 0) (layer "F.SilkS")
+      (effects (font (size 0.3 0.3) (thickness 0.05)))
     )
     (fp_line (start -0.261252 -0.735) (end 0.261252 -0.735) (layer "F.SilkS") (width 0.12))
@@
       (effects (font (size 1 1) (thickness 0.15)))
     )
-    (fp_text user "${REFERENCE}" (at 0 0 90) (layer "F.Fab")
-      (effects (font (size 0.5 0.5) (thickness 0.08)))
+    (fp_text user "${REFERENCE}" (at 0 0 90) (layer "F.SilkS")
+      (effects (font (size 0.3 0.3) (thickness 0.05)))
     )
     (fp_line (start -0.227064 0.735) (end 0.227064 0.735) (layer "F.SilkS") (width 0.12))
@@
       (effects (font (size 1 1) (thickness 0.15)))
     )
-    (fp_text user "${REFERENCE}" (at 0 0 90) (layer "F.Fab")
-      (effects (font (size 0.5 0.5) (thickness 0.08)))
+    (fp_text user "${REFERENCE}" (at 0 0 90) (layer "F.SilkS")
+      (effects (font (size 0.3 0.3) (thickness 0.05)))
     )
     (fp_line (start -0.227064 0.735) (end 0.227064 0.735) (layer "F.SilkS") (width 0.12))
@@
       (effects (font (size 1 1) (thickness 0.15)))
     )
-    (fp_text user "${REFERENCE}" (at 0 0 90) (layer "F.Fab")
-      (effects (font (size 0.5 0.5) (thickness 0.08)))
+    (fp_text user "${REFERENCE}" (at 0 0 90) (layer "F.SilkS")
+      (effects (font (size 0.3 0.3) (thickness 0.05)))
     )
     (fp_line (start -0.227064 -0.735) (end 0.227064 -0.735) (layer "F.SilkS") (width 0.12))
@@
       (effects (font (size 1 1) (thickness 0.15)))
     )
-    (fp_text user "${REFERENCE}" (at 0 0 90) (layer "F.Fab")
-      (effects (font (size 0.5 0.5) (thickness 0.08)))
+    (fp_text user "${REFERENCE}" (at 0 0 90) (layer "F.SilkS")
+      (effects (font (size 0.3 0.3) (thickness 0.05)))
     )
     (fp_line (start -0.227064 0.735) (end 0.227064 0.735) (layer "F.SilkS") (width 0.12))
@@
       (effects (font (size 1 1) (thickness 0.15)))
     )
-    (fp_text user "${REFERENCE}" (at 0 0 90) (layer "F.Fab")
-      (effects (font (size 0.5 0.5) (thickness 0.08)))
+    (fp_text user "${REFERENCE}" (at 0 0 90) (layer "F.SilkS")
+      (effects (font (size 0.3 0.3) (thickness 0.05)))
     )
     (fp_line (start -0.227064 0.735) (end 0.227064 0.735) (layer "F.SilkS") (width 0.12))
@@
       (effects (font (size 1 1) (thickness 0.15)))
     )
-    (fp_text user "${REFERENCE}" (at 0 0) (layer "F.Fab")
-      (effects (font (size 0.5 0.5) (thickness 0.08)))
+    (fp_text user "${REFERENCE}" (at 0 0) (layer "F.SilkS")
+      (effects (font (size 0.3 0.3) (thickness 0.05)))
     )
     (fp_line (start -0.261252 0.735) (end 0.261252 0.735) (layer "F.SilkS") (width 0.12))
@@
   )
   (gr_rect (start 76.2 55.88) (end 138.6332 131.4704) (layer "Edge.Cuts") (width 0.1) (fill none))
-  (gr_circle (center 79.756 59.436) (end 81.356 59.436) (layer "Edge.Cuts") (width 0.2) (fill none))
-  (gr_circle (center 134.62 128.016) (end 136.22 128.016) (layer "Edge.Cuts") (width 0.2) (fill none))
+  (gr_circle (center 79.756 59.436) (end 81.356 59.436) (layer "Edge.Cuts") (width 0.2) (fill solid))
+  (gr_circle (center 134.62 128.016) (end 136.22 128.016) (layer "Edge.Cuts") (width 0.2) (fill solid))
+  (gr_text "220" (at 110.0328 85.0392 90) (layer "F.SilkS")
+    (effects (font (size 0.5 0.5) (thickness 0.08)))
+  )
+  (gr_text "220" (at 113.7412 65.2272 90) (layer "F.SilkS")
+    (effects (font (size 0.5 0.5) (thickness 0.08)))
+  )
+  (gr_text "ControllerBox STM32F4x1\nEMCPro Firmware\n(c) Rockavoldy 2022" (at 126.3904 119.8372) (layer "F.SilkS")
+    (effects (font (size 1 1) (thickness 0.15)))
+  )
+  (gr_text "10uF" (at 119.38 63.0936 90) (layer "F.SilkS")
+    (effects (font (size 0.5 0.5) (thickness 0.08)))
+  )
+  (gr_text "10uF" (at 119.6848 84.9376 90) (layer "F.SilkS")
+    (effects (font (size 0.5 0.5) (thickness 0.08)))
+  )
+  (gr_text "10uF" (at 98.552 115.57 90) (layer "F.SilkS")
+    (effects (font (size 0.5 0.5) (thickness 0.08)))
+  )
+  (gr_text "4.7k" (at 114.6048 106.172) (layer "F.SilkS")
+    (effects (font (size 0.5 0.5) (thickness 0.08)))
+  )
+  (gr_text "220" (at 98.6028 112.3696 90) (layer "F.SilkS")
+    (effects (font (size 0.5 0.5) (thickness 0.08)))
+  )
+  (segment (start 116.84 82.7024) (end 117.3988 83.2612) (width 0.25) (layer "F.Cu") (net 2))
   (segment (start 116.3105 82.7532) (end 116.3613 82.7024) (width 0.25) (layer "F.Cu") (net 2))
   (segment (start 113.9284 82.7532) (end 116.3105 82.7532) (width 0.25) (layer "F.Cu") (net 2))
-  (segment (start 121.9748 82.7572) (end 128.4204 82.7572) (width 0.25) (layer "F.Cu") (net 2))
-  (segment (start 120.87048 81.65288) (end 121.9748 82.7572) (width 0.25) (layer "F.Cu") (net 2))
-  (segment (start 116.3613 82.7024) (end 117.41082 81.65288) (width 0.25) (layer "F.Cu") (net 2))
-  (segment (start 117.41082 81.65288) (end 120.87048 81.65288) (width 0.25) (layer "F.Cu") (net 2))
+  (segment (start 119.126 88.1888) (end 124.5576 82.7572) (width 0.25) (layer "F.Cu") (net 2))
+  (segment (start 117.3988 83.2612) (end 117.3988 87.63) (width 0.25) (layer "F.Cu") (net 2))
+  (segment (start 117.9576 88.1888) (end 119.126 88.1888) (width 0.25) (layer "F.Cu") (net 2))
+  (segment (start 124.5576 82.7572) (end 125.6832 82.7572) (width 0.25) (layer "F.Cu") (net 2))
+  (segment (start 128.4204 82.7572) (end 125.6832 82.7572) (width 0.25) (layer "F.Cu") (net 2))
+  (segment (start 117.3988 87.63) (end 117.9576 88.1888) (width 0.25) (layer "F.Cu") (net 2))
+  (segment (start 116.3613 82.7024) (end 116.84 82.7024) (width 0.25) (layer "F.Cu") (net 2))
   (segment (start 116.3105 84.709) (end 116.3613 84.7598) (width 0.25) (layer "F.Cu") (net 3))
   (segment (start 113.9284 84.709) (end 116.3105 84.709) (width 0.25) (layer "F.Cu") (net 3))
@@
   (segment (start 116.3907 84.7892) (end 128.4204 84.7892) (width 0.25) (layer "B.Cu") (net 3))
   (segment (start 113.9124 86.6648) (end 116.2089 86.6648) (width 0.25) (layer "F.Cu") (net 4))
-  (segment (start 128.4204 86.8212) (end 121.8652 86.8212) (width 0.25) (layer "F.Cu") (net 4))
-  (segment (start 117.41082 87.86672) (end 120.81968 87.86672) (width 0.25) (layer "F.Cu") (net 4))
-  (segment (start 116.3613 86.8172) (end 117.41082 87.86672) (width 0.25) (layer "F.Cu") (net 4))
+  (segment (start 120.04808 88.63832) (end 121.8652 86.8212) (width 0.25) (layer "F.Cu") (net 4))
+  (segment (start 116.3613 87.228217) (end 117.771403 88.63832) (width 0.25) (layer "F.Cu") (net 4))
+  (segment (start 117.771403 88.63832) (end 120.04808 88.63832) (width 0.25) (layer "F.Cu") (net 4))
   (segment (start 116.2089 86.6648) (end 116.3613 86.8172) (width 0.25) (layer "F.Cu") (net 4))
-  (segment (start 120.81968 87.86672) (end 121.8652 86.8212) (width 0.25) (layer "F.Cu") (net 4))
+  (segment (start 121.8652 86.8212) (end 128.4204 86.8212) (width 0.25) (layer "F.Cu") (net 4))
+  (segment (start 116.3613 86.8172) (end 116.3613 87.228217) (width 0.25) (layer "F.Cu") (net 4))
   (segment (start 128.4204 65.1764) (end 117.5004 65.1764) (width 0.25) (layer "F.Cu") (net 5))
   (segment (start 117.5004 65.1764) (end 117.4496 65.2272) (width 0.25) (layer "F.Cu") (net 5))
@@
   (segment (start 104.7844 109.5088) (end 96.9772 101.7016) (width 0.25) (layer "F.Cu") (net 19))
   (segment (start 114.6048 109.5088) (end 112.6236 109.5088) (width 0.25) (layer "F.Cu") (net 19))
+  (segment (start 91.5416 101.7016) (end 92.9132 101.7016) (width 0.25) (layer "B.Cu") (net 19))
+  (segment (start 96.012 69.2912) (end 106.7816 58.5216) (width 0.25) (layer "B.Cu") (net 19))
+  (segment (start 96.012 98.6028) (end 96.012 69.2912) (width 0.25) (layer "B.Cu") (net 19))
+  (segment (start 92.9132 101.7016) (end 96.012 98.6028) (width 0.25) (layer "B.Cu") (net 19))
   (segment (start 126.9004 103.886) (end 128.4204 102.366) (width 0.25) (layer "F.Cu") (net 20))
   (segment (start 112.6236 107.5088) (end 116.2464 103.886) (width 0.25) (layer "F.Cu") (net 20))
@@
   (segment (start 106.7816 89.0016) (end 116.586 98.806) (width 0.25) (layer "B.Cu") (net 22))
   (segment (start 116.586 98.806) (end 116.586 107.5088) (width 0.25) (layer "B.Cu") (net 22))
+  (via (at 111.9284 82.7532) (size 0.8) (drill 0.4) (layers "F.Cu" "B.Cu") (net 23))
+  (segment (start 106.7816 86.4616) (end 110.49 82.7532) (width 0.25) (layer "B.Cu") (net 23))
+  (segment (start 110.49 82.7532) (end 111.9284 82.7532) (width 0.25) (layer "B.Cu") (net 23))
+  (segment (start 111.9284 84.709) (end 111.141 83.9216) (width 0.25) (layer "F.Cu") (net 24))
+  (segment (start 111.141 83.9216) (end 106.7816 83.9216) (width 0.25) (layer "F.Cu") (net 24))
+  (segment (start 112.169293 81.3816) (end 112.9284 82.140707) (width 0.25) (layer "F.Cu") (net 25))
+  (segment (start 106.7816 81.3816) (end 112.169293 81.3816) (width 0.25) (layer "F.Cu") (net 25))
+  (segment (start 112.9284 82.140707) (end 112.9284 85.6488) (width 0.25) (layer "F.Cu") (net 25))
+  (segment (start 112.9284 85.6488) (end 111.9124 86.6648) (width 0.25) (layer "F.Cu") (net 25))
   (segment (start 109.3724 68.3768) (end 109.3724 76.2508) (width 0.25) (layer "F.Cu") (net 26))
   (segment (start 110.506 67.2432) (end 109.3724 68.3768) (width 0.25) (layer "F.Cu") (net 26))

Commit message: add readme; fix wrong pin issue for G29Shifter
Parts:
- HBRAKE1: value HAND BRAKE -> RJ45
- J1: value ROW BUTTON -> Conn_01x05_Male
- J2: value COL BUTTON -> Conn_01x04_Male
- PEDAL1: value PEDAL -> RJ45
- STEERINGWHEEL1: value STEERING WHEEL -> RJ45
- renumbered G29SHIFTER to G29SHIFTER1
Connections:
- G29SHIFTER1 pad 6: unconnected-(G29SHIFTER1-Pad6) -> GND
- G29SHIFTER1 pad 7: SHIFTER Y -> VCC 3.3V
- G29SHIFTER1 pad 8: VCC 3.3V -> SHIFTER Y
- G29SHIFTER1 pad 9: GND -> unconnected-(G29SHIFTER1-Pad9)
Routing:
- net VCC 3.3V: track 130.5 -> 136.0 mm
- net SHIFTER Y: track 9.98 -> 11.1 mm
